File: KiCad/UWBkit_sniffer/UWBkit_sniffer.kicad_sch (KiCad schematic)
At the start: 11 parts, among them J1 Conn_I2C1, J2 Conn_I2C2, J3 Conn_01x03, J4 Conn_SPIS, J5 Conn_SPIM

Commit message: Release V1.0
Changed lines of the file:
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@@
 	(title_block
 		(title "UWBkit - UWB Sniffer")
-		(date "2025-12-15")
-		(rev "1")
+		(date "2026-02-24")
+		(rev "1.0")
 	)
 	(text "Remove if\nflow control\nis UNUSED"
@@
 		)
 	)
-	(text_box "UWC.20\nUWA.01\nI-PEX MHF I connector\nSMA connector\n\nsensniff\n"
-		(exclude_from_sim no)
-		(at 240.03 19.05 0)
-		(size 36.83 46.99)
-		(margins 0.9525 0.9525 0.9525 0.9525)
-		(stroke
-			(width 0)
-			(type solid)
-		)
-		(fill
-			(type none)
-		)
-		(effects
-			(font
-				(size 1.27 1.27)
-			)
-			(justify left top)
-		)
-	)
